File: pcb/lk16c-pcb.kicad_pcb (KiCad board)
At the start: 2 copper layers, 76.2 x 76.2 mm, 53 parts, among them J1 Conn_01x04, J2 Conn_01x04, J3 Conn_01x04, J4 Conn_01x04, J5 Conn_01x04, J6 Conn_01x04, J7 PINHD_1x03_ARGB, J8 PINHD_1x05_I2C, SW1 SW_Push, SW10 SW_Push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

Commit message: Move Fab DataMatrix footprint
Parts:
- moved TXT1 1.27 mm to (85.7, 78.7)
Changed lines of the file:
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@@
 	(footprint "LKBD_PCBFab:JLCPCB_2DBarcode_5x5mm"
 		(layer "B.Cu")
-		(at 85.725 80.01 180)
+		(at 85.725 78.74 180)
 		(descr "2D barcode (5 × 5 mm) placeholder for JLCPCB")
 		(tags "JLCPCB 2DBarcode")
